File: M-O-Y/M-O-Y.kicad_pcb (KiCad board)
At the start: 2 copper layers, 165 x 94 mm, 9 parts, among them U1 ESP32-S3-DEVKITC-1-N8R2, U10 AMS1117-3.3, U8 Step_Down +5v

Commit message: PCB
Parts:
- added G***: LOGO, LOGO, F.Cu at (119.0, 106.0)
Other:
- board text added: "Made By Youssef Ayman"
